Commit message: pipeline

File: body4.urdf (robot description, URDF)
Before this commit: robot robot, 2 links, 1 joints
Links:
- removed link Central
- removed link FrontOne
- added link half0half, mass 1; collision mesh filename=RhomDoDeca_mm v9.stl scale=0.1 0.1 0.1; visual mesh filename=RhomDoDeca_mm v9.stl scale=0.1 0.1 0.1
- added link half1half, mass 1; collision mesh filename=RhomDoDeca_mm v9.stl scale=0.1 0.1 0.1; visual mesh filename=RhomDoDeca_mm v9.stl scale=0.1 0.1 0.1
- added link half2half, mass 1; collision mesh filename=RhomDoDeca_mm v9.stl scale=0.1 0.1 0.1; visual mesh filename=RhomDoDeca_mm v9.stl scale=0.1 0.1 0.1
- added link half3half, mass 1; collision mesh filename=RhomDoDeca_mm v9.stl scale=0.1 0.1 0.1; visual mesh filename=RhomDoDeca_mm v9.stl scale=0.1 0.1 0.1
- added link one0, mass 1; collision mesh filename=RhomDoDeca_mm v9.stl scale=0.1 0.1 0.1; visual mesh filename=RhomDoDeca_mm v9.stl scale=0.1 0.1 0.1
- added link one1, mass 1; collision mesh filename=RhomDoDeca_mm v9.stl scale=0.1 0.1 0.1; visual mesh filename=RhomDoDeca_mm v9.stl scale=0.1 0.1 0.1
- added link zero0, mass 1; collision mesh filename=RhomDoDeca_mm v9.stl scale=0.1 0.1 0.1; visual mesh filename=RhomDoDeca_mm v9.stl scale=0.1 0.1 0.1
- added link zero1, mass 1; collision mesh filename=RhomDoDeca_mm v9.stl scale=0.1 0.1 0.1; visual mesh filename=RhomDoDeca_mm v9.stl scale=0.1 0.1 0.1
- added link zero2, mass 1; collision mesh filename=RhomDoDeca_mm v9.stl scale=0.1 0.1 0.1; visual mesh filename=RhomDoDeca_mm v9.stl scale=0.1 0.1 0.1
- added link zero3, mass 1; collision mesh filename=RhomDoDeca_mm v9.stl scale=0.1 0.1 0.1; visual mesh filename=RhomDoDeca_mm v9.stl scale=0.1 0.1 0.1
Joints:
- removed joint Central_FrontOne
- added joint half0half_one0: type fixed, parent half0half, child one0, origin xyz=2.88 2.043 -2.043 rpy=0 0 0, axis 0 1 0, limit lower=-3.14159 upper=3.14159 effort=0.0 velocity=0.0
- added joint half1half_half0half: type fixed, parent half1half, child half0half, origin xyz=0 -4.086 0 rpy=0 0 0, axis 0 1 0, limit lower=-3.14159 upper=3.14159 effort=0.0 velocity=0.0
- added joint half2half_half1half: type fixed, parent half2half, child half1half, origin xyz=0 -4.086 0 rpy=0 0 0, axis 0 1 0, limit lower=-3.14159 upper=3.14159 effort=0.0 velocity=0.0
- added joint half3half_half2half: type fixed, parent half3half, child half2half, origin xyz=0 -4.086 0 rpy=0 0 0, axis 0 1 0, limit lower=-3.14159 upper=3.14159 effort=0.0 velocity=0.0
- added joint one0_one1: type fixed, parent one0, child one1, origin xyz=0 4.086 0 rpy=0 0 0, axis 0 1 0, limit lower=-3.14159 upper=3.14159 effort=0.0 velocity=0.0
- added joint zero0_zero1: type fixed, parent zero0, child zero1, origin xyz=0 4.086 0 rpy=0 0 0, axis 0 1 0, limit lower=-3.14159 upper=3.14159 effort=0.0 velocity=0.0
- added joint zero1_zero2: type fixed, parent zero1, child zero2, origin xyz=0 4.086 0 rpy=0 0 0, axis 0 1 0, limit lower=-3.14159 upper=3.14159 effort=0.0 velocity=0.0
- added joint zero2_zero3: type fixed, parent zero2, child zero3, origin xyz=0 4.086 0 rpy=0 0 0, axis 0 1 0, limit lower=-3.14159 upper=3.14159 effort=0.0 velocity=0.0
- added joint zero3_half3half: type fixed, parent zero3, child half3half, origin xyz=2.88 -2.043 2.043 rpy=0 0 0, axis 0 1 0, limit lower=-3.14159 upper=3.14159 effort=0.0 velocity=0.0
